File: electronics/mainboard/mainboard.sch (EAGLE design)
At the start: 67 parts, among them CON1 B3B-ZR, IC1 TPS6300, IC2 TPS77033, J1 2MMPAD, J10 2MMPAD, J11 ROUND1MM, J12 ROUND1MM, J13 ROUND1MM, J14 ROUND1MM, J15 ROUND1MM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

Commit message: changed crystal.  name change.  minor tweaks
Parts:
- Q1: device SparkFun-FreqCtrl:CRYSTAL-GROUNDED -> crystals:25MHZ-3X2MM
Connections:
- net GND: now also Q1.2; no longer Q1.3
- net N$15: now also Q1.3; no longer Q1.2
Changed lines of the file:
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@@
 <grid distance="0.1" unitdist="inch" unit="inch" style="lines" multiple="1" display="no" altdistance="0.01" altunitdist="inch" altunit="inch"/>
 <layers>
-<layer number="1" name="Top" color="4" fill="1" visible="no" active="no"/>
-<layer number="16" name="Bottom" color="1" fill="1" visible="no" active="no"/>
-<layer number="17" name="Pads" color="2" fill="1" visible="no" active="no"/>
-<layer number="18" name="Vias" color="2" fill="1" visible="no" active="no"/>
-<layer number="19" name="Unrouted" color="6" fill="1" visible="no" active="no"/>
-<layer number="20" name="Dimension" color="15" fill="1" visible="no" active="no"/>
-<layer number="21" name="tPlace" color="7" fill="1" visible="no" active="no"/>
-<layer number="22" name="bPlace" color="7" fill="1" visible="no" active="no"/>
-<layer number="23" name="tOrigins" color="15" fill="1" visible="no" active="no"/>
-<layer number="24" name="bOrigins" color="15" fill="1" visible="no" active="no"/>
-<layer number="25" name="tNames" color="7" fill="1" visible="no" active="no"/>
-<layer number="26" name="bNames" color="7" fill="1" visible="no" active="no"/>
-<layer number="27" name="tValues" color="7" fill="1" visible="no" active="no"/>
-<layer number="28" name="bValues" color="7" fill="1" visible="no" active="no"/>
+<layer number="1" name="Top" color="4" fill="1" visible="yes" active="no"/>
+<layer number="16" name="Bottom" color="1" fill="1" visible="yes" active="no"/>
+<layer number="17" name="Pads" color="2" fill="1" visible="yes" active="no"/>
+<layer number="18" name="Vias" color="2" fill="1" visible="yes" active="no"/>
+<layer number="19" name="Unrouted" color="6" fill="1" visible="yes" active="no"/>
+<layer number="20" name="Dimension" color="15" fill="1" visible="yes" active="no"/>
+<layer number="21" name="tPlace" color="7" fill="1" visible="yes" active="no"/>
+<layer number="22" name="bPlace" color="7" fill="1" visible="yes" active="no"/>
+<layer number="23" name="tOrigins" color="15" fill="1" visible="yes" active="no"/>
+<layer number="24" name="bOrigins" color="15" fill="1" visible="yes" active="no"/>
+<layer number="25" name="tNames" color="7" fill="1" visible="yes" active="no"/>
+<layer number="26" name="bNames" color="7" fill="1" visible="yes" active="no"/>
+<layer number="27" name="tValues" color="7" fill="1" visible="yes" active="no"/>
+<layer number="28" name="bValues" color="7" fill="1" visible="yes" active="no"/>
 <layer number="29" name="tStop" color="7" fill="3" visible="no" active="no"/>
 <layer number="30" name="bStop" color="7" fill="6" visible="no" active="no"/>
@@
 <layer number="35" name="tGlue" color="7" fill="4" visible="no" active="no"/>
 <layer number="36" name="bGlue" color="7" fill="5" visible="no" active="no"/>
-<layer number="37" name="tTest" color="7" fill="1" visible="no" active="no"/>
-<layer number="38" name="bTest" color="7" fill="1" visible="no" active="no"/>
+<layer number="37" name="tTest" color="7" fill="1" visible="yes" active="no"/>
+<layer number="38" name="bTest" color="7" fill="1" visible="yes" active="no"/>
 <layer number="39" name="tKeepout" color="4" fill="11" visible="no" active="no"/>
 <layer number="40" name="bKeepout" color="1" fill="11" visible="no" active="no"/>
@@
 <layer number="44" name="Drills" color="7" fill="1" visible="no" active="no"/>
 <layer number="45" name="Holes" color="7" fill="1" visible="no" active="no"/>
-<layer number="46" name="Milling" color="3" fill="1" visible="no" active="no"/>
-<layer number="47" name="Measures" color="7" fill="1" visible="no" active="no"/>
-<layer number="48" name="Document" color="7" fill="1" visible="no" active="no"/>
-<layer number="49" name="Reference" color="7" fill="1" visible="no" active="no"/>
-<layer number="50" name="dxf" color="7" fill="1" visible="no" active="no"/>
-<layer number="51" name="tDocu" color="7" fill="1" visible="no" active="no"/>
-<layer number="52" name="bDocu" color="7" fill="1" visible="no" active="no"/>
-<layer number="53" name="tGND_GNDA" color="7" fill="9" visible="no" active="no"/>
-<layer number="54" name="bGND_GNDA" color="1" fill="9" visible="no" active="no"/>
-<layer number="56" name="wert" color="7" fill="1" visible="no" active="no"/>
-<layer number="57" name="tCAD" color="7" fill="1" visible="no" active="no"/>
+<layer number="46" name="Milling" color="3" fill="1" visible="yes" active="no"/>
+<layer number="47" name="Measures" color="7" fill="1" visible="yes" active="no"/>
+<layer number="48" name="Document" color="7" fill="1" visible="yes" active="no"/>
+<layer number="49" name="Reference" color="7" fill="1" visible="yes" active="no"/>
+<layer number="50" name="dxf" color="7" fill="1" visible="yes" active="no"/>
+<layer number="51" name="tDocu" color="7" fill="1" visible="yes" active="no"/>
+<layer number="52" name="bDocu" color="7" fill="1" visible="yes" active="no"/>
+<layer number="53" name="tGND_GNDA" color="7" fill="9" visible="yes" active="no"/>
+<layer number="54" name="bGND_GNDA" color="1" fill="9" visible="yes" active="no"/>
+<layer number="56" name="wert" color="7" fill="1" visible="yes" active="no"/>
+<layer number="57" name="tCAD" color="7" fill="1" visible="yes" active="no"/>
+<layer number="90" name="Modules" color="5" fill="1" visible="yes" active="yes"/>
 <layer number="91" name="Nets" color="2" fill="1" visible="yes" active="yes"/>
 <layer number="92" name="Busses" color="1" fill="1" visible="yes" active="yes"/>
@@
 <part name="J8" library="connectors" deviceset="2MMPAD" device=""/>
 <part name="J9" library="connectors" deviceset="2MMPAD" device=""/>
-<part name="Q1" library="SparkFun-FreqCtrl" deviceset="CRYSTAL-GROUNDED" device="" value="25Mhz"/>
+<part name="Q1" library="crystals" deviceset="25MHZ-3X2MM" device="" value="25Mhz"/>
 <part name="SUPPLY38" library="supply2" deviceset="GND" device=""/>
 <part name="C20" library="rcl" deviceset="C-US" device="C0603" value="18pf"/>
@@
 </segment>
 <segment>
-<pinref part="Q1" gate="G$1" pin="3"/>
-<pinref part="SUPPLY38" gate="GND" pin="GND"/>
-</segment>
-<segment>
 <pinref part="C20" gate="G$1" pin="2"/>
 <pinref part="SUPPLY39" gate="GND" pin="GND"/>
@@
 <pinref part="U2" gate="A" pin="VBUS"/>
 <pinref part="SUPPLY47" gate="GND" pin="GND"/>
+</segment>
+<segment>
+<pinref part="SUPPLY38" gate="GND" pin="GND"/>
+<pinref part="Q1" gate="G$1" pin="2"/>
 </segment>
 </net>
@@
 <wire x1="116.84" y1="-5.08" x2="147.32" y2="-5.08" width="0.1524" layer="91"/>
 <wire x1="147.32" y1="-5.08" x2="147.32" y2="0" width="0.1524" layer="91"/>
-<pinref part="Q1" gate="G$1" pin="2"/>
 <wire x1="147.32" y1="0" x2="152.4" y2="0" width="0.1524" layer="91"/>
 <pinref part="C20" gate="G$1" pin="1"/>
+<pinref part="Q1" gate="G$1" pin="3"/>
+<wire x1="152.4" y1="-2.54" x2="152.4" y2="0" width="0.1524" layer="91"/>
 <junction x="152.4" y="0"/>
-<wire x1="152.4" y1="0" x2="152.4" y2="-2.54" width="0.1524" layer="91"/>
-</segment>
-</net>
+</segment>
+</net>

Commit message: minor changes for board production.  REV0 off to board house
Parts:
- added J17, J18, J19, J20: ROUND1MM, connectors:ROUND1MM
Connections:
- new net N$29: J17.P$1, U2.P4.7/PM_NONE
- new net N$30: J18.P$1, U2.P4.6/PM_NONE
- new net N$31: J19.P$1, U2.PU.0/DP
- new net N$32: J20.P$1, U2.PU.1/DM
Other:
- moved on the sheet: C20, C21, C22, R12
Changed lines of the file:
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@@
 <part name="J15" library="connectors" deviceset="ROUND1MM" device=""/>
 <part name="J16" library="connectors" deviceset="ROUND1MM" device=""/>
+<part name="J17" library="connectors" deviceset="ROUND1MM" device=""/>
+<part name="J18" library="connectors" deviceset="ROUND1MM" device=""/>
+<part name="J19" library="connectors" deviceset="ROUND1MM" device=""/>
+<part name="J20" library="connectors" deviceset="ROUND1MM" device=""/>
 </parts>
 <sheets>
@@
 <attribute name="NAME" x="-10.16" y="109.22" size="1.778" layer="95" rot="R180"/>
 </instance>
-<instance part="Q1" gate="G$1" x="152.4" y="-5.08" smashed="yes" rot="R90">
-<attribute name="VALUE" x="149.86" y="-7.62" size="1.778" layer="96" rot="R90"/>
-</instance>
-<instance part="SUPPLY38" gate="GND" x="160.02" y="-5.08" smashed="yes" rot="R90"/>
-<instance part="C20" gate="G$1" x="154.94" y="0" smashed="yes" rot="R90">
-<attribute name="NAME" x="154.305" y="1.016" size="1.778" layer="95" rot="R90"/>
-<attribute name="VALUE" x="159.131" y="1.016" size="1.778" layer="96" rot="R90"/>
-</instance>
-<instance part="C21" gate="G$1" x="154.94" y="-10.16" smashed="yes" rot="R90">
-<attribute name="NAME" x="152.273" y="-11.176" size="1.778" layer="95" rot="R270"/>
-<attribute name="VALUE" x="157.861" y="-11.43" size="1.778" layer="96" rot="R270"/>
-</instance>
-<instance part="SUPPLY39" gate="GND" x="162.56" y="0" smashed="yes" rot="R90">
-<attribute name="VALUE" x="165.989" y="-5.461" size="1.778" layer="96" rot="R90"/>
-</instance>
-<instance part="SUPPLY40" gate="GND" x="162.56" y="-10.16" smashed="yes" rot="R90"/>
+<instance part="Q1" gate="G$1" x="160.02" y="-5.08" smashed="yes" rot="R90">
+<attribute name="VALUE" x="157.48" y="-7.62" size="1.778" layer="96" rot="R90"/>
+</instance>
+<instance part="SUPPLY38" gate="GND" x="167.64" y="-5.08" smashed="yes" rot="R90"/>
+<instance part="C20" gate="G$1" x="162.56" y="0" smashed="yes" rot="R90">
+<attribute name="NAME" x="161.925" y="1.016" size="1.778" layer="95" rot="R90"/>
+<attribute name="VALUE" x="166.751" y="1.016" size="1.778" layer="96" rot="R90"/>
+</instance>
+<instance part="C21" gate="G$1" x="162.56" y="-10.16" smashed="yes" rot="R90">
+<attribute name="NAME" x="159.893" y="-11.176" size="1.778" layer="95" rot="R270"/>
+<attribute name="VALUE" x="165.481" y="-11.43" size="1.778" layer="96" rot="R270"/>
+</instance>
+<instance part="SUPPLY39" gate="GND" x="170.18" y="0" smashed="yes" rot="R90">
+<attribute name="VALUE" x="173.609" y="-5.461" size="1.778" layer="96" rot="R90"/>
+</instance>
+<instance part="SUPPLY40" gate="GND" x="170.18" y="-10.16" smashed="yes" rot="R90"/>
 <instance part="R6" gate="G$1" x="243.84" y="60.96" smashed="yes" rot="R90">
 <attribute name="NAME" x="242.3414" y="57.15" size="1.778" layer="95" rot="R90"/>
@@
 <attribute name="VALUE" x="247.142" y="-22.86" size="1.778" layer="96" rot="R90"/>
 </instance>
-<instance part="SUPPLY41" gate="GND" x="142.24" y="-2.54" smashed="yes" rot="R90"/>
-<instance part="C22" gate="G$1" x="139.7" y="2.54"/>
-<instance part="R12" gate="G$1" x="139.7" y="10.16" smashed="yes" rot="R270">
-<attribute name="NAME" x="141.1986" y="13.97" size="1.778" layer="95" rot="R270"/>
-<attribute name="VALUE" x="141.478" y="8.89" size="1.778" layer="96" rot="R270"/>
-</instance>
-<instance part="+3V5" gate="G$1" x="139.7" y="17.78"/>
+<instance part="SUPPLY41" gate="GND" x="149.86" y="-2.54" smashed="yes" rot="R90"/>
+<instance part="C22" gate="G$1" x="147.32" y="2.54"/>
+<instance part="R12" gate="G$1" x="147.32" y="10.16" smashed="yes" rot="R270">
+<attribute name="NAME" x="148.8186" y="13.97" size="1.778" layer="95" rot="R270"/>
+<attribute name="VALUE" x="149.098" y="8.89" size="1.778" layer="96" rot="R270"/>
+</instance>
+<instance part="+3V5" gate="G$1" x="147.32" y="17.78"/>
 <instance part="U5" gate="G$1" x="213.36" y="114.3"/>
 <instance part="SUPPLY44" gate="GND" x="195.58" y="99.06"/>
@@
 <instance part="J15" gate="G$1" x="10.16" y="-15.24" rot="R180"/>
 <instance part="J16" gate="G$1" x="25.4" y="2.54" rot="R180"/>
+<instance part="J17" gate="G$1" x="121.92" y="5.08"/>
+<instance part="J18" gate="G$1" x="121.92" y="7.62"/>
+<instance part="J19" gate="G$1" x="121.92" y="-43.18"/>
+<instance part="J20" gate="G$1" x="121.92" y="-45.72"/>
 </instances>
 <busses>
@@
 <pinref part="U2" gate="A" pin="P5.1"/>
 <pinref part="SUPPLY41" gate="GND" pin="GND"/>
-<wire x1="116.84" y1="-2.54" x2="139.7" y2="-2.54" width="0.1524" layer="91"/>
+<wire x1="116.84" y1="-2.54" x2="147.32" y2="-2.54" width="0.1524" layer="91"/>
 <pinref part="C22" gate="G$1" pin="2"/>
-<junction x="139.7" y="-2.54"/>
+<junction x="147.32" y="-2.54"/>
 </segment>
 <segment>
@@
 <segment>
 <pinref part="U2" gate="A" pin="P4.5/PM_UCA1RXD/PM_UCA1SOMI"/>
-<wire x1="116.84" y1="10.16" x2="121.92" y2="10.16" width="0.1524" layer="91"/>
-<label x="121.92" y="10.16" size="1.778" layer="95"/>
+<wire x1="116.84" y1="10.16" x2="124.46" y2="10.16" width="0.1524" layer="91"/>
+<label x="124.46" y="10.16" size="1.778" layer="95"/>
 </segment>
 </net>
@@
 <segment>
 <pinref part="U2" gate="A" pin="P5.2/XT2IN"/>
-<wire x1="116.84" y1="-5.08" x2="147.32" y2="-5.08" width="0.1524" layer="91"/>
-<wire x1="147.32" y1="-5.08" x2="147.32" y2="0" width="0.1524" layer="91"/>
-<wire x1="147.32" y1="0" x2="152.4" y2="0" width="0.1524" layer="91"/>
+<wire x1="116.84" y1="-5.08" x2="154.94" y2="-5.08" width="0.1524" layer="91"/>
+<wire x1="154.94" y1="-5.08" x2="154.94" y2="0" width="0.1524" layer="91"/>
+<wire x1="154.94" y1="0" x2="160.02" y2="0" width="0.1524" layer="91"/>
 <pinref part="C20" gate="G$1" pin="1"/>
 <pinref part="Q1" gate="G$1" pin="3"/>
-<wire x1="152.4" y1="-2.54" x2="152.4" y2="0" width="0.1524" layer="91"/>
-<junction x="152.4" y="0"/>
+<wire x1="160.02" y1="-2.54" x2="160.02" y2="0" width="0.1524" layer="91"/>
+<junction x="160.02" y="0"/>
 </segment>
 </net>
@@
 <pinref part="U2" gate="A" pin="P5.3/XT2OUT"/>
 <pinref part="Q1" gate="G$1" pin="1"/>
-<wire x1="116.84" y1="-7.62" x2="152.4" y2="-7.62" width="0.1524" layer="91"/>
+<wire x1="116.84" y1="-7.62" x2="160.02" y2="-7.62" width="0.1524" layer="91"/>
 <pinref part="C21" gate="G$1" pin="1"/>
-<wire x1="152.4" y1="-10.16" x2="152.4" y2="-7.62" width="0.1524" layer="91"/>
-<junction x="152.4" y="-7.62"/>
+<wire x1="160.02" y1="-10.16" x2="160.02" y2="-7.62" width="0.1524" layer="91"/>
+<junction x="160.02" y="-7.62"/>
 </segment>
 </net>
@@
 <segment>
 <pinref part="U2" gate="A" pin="P5.0"/>
-<wire x1="116.84" y1="0" x2="119.38" y2="0" width="0.1524" layer="91"/>
+<wire x1="116.84" y1="0" x2="127" y2="0" width="0.1524" layer="91"/>
 <pinref part="C22" gate="G$1" pin="1"/>
-<wire x1="139.7" y1="5.08" x2="119.38" y2="5.08" width="0.1524" layer="91"/>
-<wire x1="119.38" y1="5.08" x2="119.38" y2="0" width="0.1524" layer="91"/>
+<wire x1="147.32" y1="5.08" x2="127" y2="5.08" width="0.1524" layer="91"/>
+<wire x1="127" y1="5.08" x2="127" y2="0" width="0.1524" layer="91"/>
 <pinref part="R12" gate="G$1" pin="2"/>
-<junction x="139.7" y="5.08"/>
+<junction x="147.32" y="5.08"/>
 </segment>
 </net>
@@
 </segment>
 </net>
+<net name="N$29" class="0">
+<segment>
+<pinref part="U2" gate="A" pin="P4.7/PM_NONE"/>
+<pinref part="J17" gate="G$1" pin="P$1"/>
+</segment>
+</net>
+<net name="N$30" class="0">
+<segment>
+<pinref part="U2" gate="A" pin="P4.6/PM_NONE"/>
+<pinref part="J18" gate="G$1" pin="P$1"/>
+</segment>
+</net>
+<net name="N$31" class="0">
+<segment>
+<pinref part="U2" gate="A" pin="PU.0/DP"/>
+<pinref part="J19" gate="G$1" pin="P$1"/>
+</segment>
+</net>
+<net name="N$32" class="0">
+<segment>
+<pinref part="U2" gate="A" pin="PU.1/DM"/>
+<pinref part="J20" gate="G$1" pin="P$1"/>
+</segment>
+</net>
